File: DatatrakEPROMEmu.brd (EAGLE design)
At the start: 151.1 x 58.1 mm, 46 parts, among them IC1 LD1117AS33TR, IC2 XC95144XL_TQ144_P, Q1 BC847CSMD, Q2 BC847CSMD, Q3 BC847CSMD, U1 SN74LVCH16T245DGGR, U2 SN74LVCH16T245DGGR, U3 SN74LVCH16T245DGGR, U4 IS62WV25616DBLL-45TLI, U5 FT240XS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

Commit message: add missing D_LV8 net between CPLD and SRAM/translator
OSHPark PCBs had a missing net -- D_LV8 -- the 8th data bit from the level
translator to the CPLD. These boards will need a greenwire.
Connections:
- net D_LV8: now also IC2.135
Changed lines of the file:
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@@
 <wire x1="50.1879" y1="36.7538" x2="52.1462" y2="36.7538" width="0.1524" layer="1"/>
 <wire x1="34.163" y1="38.354" x2="35.2172" y2="38.354" width="0.1524" layer="1"/>
+<contactref element="IC2" pad="135"/>
+<wire x1="52.1462" y1="36.7538" x2="89.095" y2="46.895" width="0" layer="19" extent="1-1"/>
 </signal>
 <signal name="D_LV9">

Commit message: Route missing D_LV8 net, bump to Rev B
Routing:
- net D_LV8: track 18.7 -> 71.4 mm, vias 0 -> 2
Other:
- board text added: "DATATRAK LOCATOR Mk.II ROM CARTRIDGE EMULATOR REV B 2016-11-16 PAP"
- board text removed: "DATATRAK LOCATOR Mk.II ROM CARTRIDGE EMULATOR REV A 2016-11-14 PAP"
